Commit message: lidar and cmdvel test pass

File: lite3_description/xacro/imu_link.xacro (robot description, xacro)
@@ -4,5 +4,5 @@
     <parent link="TORSO"/>
     <child link="imu_link"/>
-    <origin rpy="0 0 0" xyz="0 0 0"/>
+    <origin rpy="0 0 0" xyz="0.05 0 0"/>
   </joint>
   <link name="imu_link">
