Commit message: add fast lio launch

File: lite3_description/xacro/body.xacro (robot description, xacro)
@@ -3,5 +3,5 @@
   <xacro:property name="damping" value="0.1"/>
   <xacro:property name="friction" value="0.1"/>
-  <xacro:include filename="$(find lite3_description)/xacro/imu_link.xacro"/>
+  <xacro:include filename="perception.xacro"/>
   <link name="base">
     <visual>

File: lite3_description/xacro/perception.xacro (robot description, xacro)
@@ -25,3 +25,29 @@
     </collision>
   </link>
+  <joint name="laser_joint" type="fixed">
+    <parent link="TORSO"/>
+    <child link="laser_link"/>
+    <origin rpy="0 0 1.57" xyz="0.163 0 0.058"/>
+  </joint>
+  <link name="laser_link">
+    <visual>
+      <origin rpy="0 0 0" xyz="0 0 0"/>
+      <geometry>
+        <box size="0.001 0.001 0.001"/>
+      </geometry>
+    </visual>
+  </link>
+  <joint name="body_joint" type="fixed">
+    <parent link="TORSO"/>
+    <child link="body"/>
+    <origin rpy="0 0 1.57" xyz="0 0 0"/>
+  </joint>
+  <link name="body">
+    <visual>
+      <origin rpy="0 0 0" xyz="0 0 0"/>
+      <geometry>
+        <box size="0.001 0.001 0.001"/>
+      </geometry>
+    </visual>
+  </link>
 </robot>

File: lite3_description/xacro/robot.xacro (robot description, xacro)
@@ -1,6 +1,6 @@
 <?xml version="1.0"?>
 <robot name="lite3" xmlns:xacro="http://www.ros.org/wiki/xacro">
-  <xacro:include filename="$(find lite3_description)/xacro/body.xacro"/>
-  <xacro:include filename="$(find lite3_description)/xacro/transmission.xacro"/>
+  <xacro:include filename="body.xacro"/>
+  <xacro:include filename="transmission.xacro"/>
   <xacro:arg name="GAZEBO" default="false"/>
   <xacro:arg name="CLASSIC" default="false"/>
